File: spar_sensor/spar_sensor.kicad_pcb (KiCad board)
At the start: 2 copper layers, 39.8 x 21.5 mm, 24 parts, among them J1 Conn_01x03_Pin, J2 Conn_01x04_Pin, J3 Conn_01x04_Pin, J4 AVR-ISP-6, Q1 MMS8550, Q2 2N7002K, SW1 SW_DPST_x2, U1 HX711, U2 ATtiny85-20M

Commit message: Touched up spar sensor to reflect parts as ordered
Parts:
- C1, C2: value 10 u -> 10u
- C3, C4, C5: value 0.1 u -> 0.1u
- Q1: value MMS8550 -> MMBT2907
- R2: value 5 k -> 5.1k
- R4, R6: value 10 k -> 10k
- R5: value 5.6 k -> 5.6k

Commit message: Updated spar sensor to reflect order
Parts:
- Q1: value MMBT2907 -> MMSS8550
- R2: value 5.1k -> 5.6k
Changed lines of the file:
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@@
         (effects (font (size 1 1) (thickness 0.15)))
     )
-    (fp_text value "MMBT2907" (at 0 2.4) (layer "F.Fab")
+    (fp_text value "MMSS8550" (at 0 2.4) (layer "F.Fab")
         (effects (font (size 1 1) (thickness 0.15)))
     )
@@
         (effects (font (size 1 1) (thickness 0.15)))
     )
-    (fp_text value "5.1k" (at 0 1.43 90) (layer "F.Fab")
+    (fp_text value "5.6k" (at 0 1.43 90) (layer "F.Fab")
         (effects (font (size 1 1) (thickness 0.15)))
     )
