File: servo_regulator/servo_regulator.kicad_pcb (KiCad board)
At the start: 2 copper layers, 17 x 15.6 mm, 18 parts, among them J1 Conn_01x03_Socket, Q1 2N7002K, Q2 2N7002K

Commit message: Updated spar sensor to reflect order
Parts:
- R4, R5: value 420 -> 430
- U1: value ~ -> TPS563208DDCR
Changed lines of the file:
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@@
     (descr "Capacitor SMD 0805 (2012 Metric), square (rectangular) end terminal, IPC_7351 nominal, (Body size source: IPC-SM-782 page 76, https://www.pcb-3d.com/wordpress/wp-content/uploads/ipc-sm-782a_amendment_1_and_2.pdf, https://docs.google.com/spreadsheets/d/1BsfQQcO9C6DZCsRaXUlFlo91Tg2WpOkGARC1WS5S8t0/edit?usp=sharing), generated with kicad-footprint-generator")
     (tags "capacitor")
-    (property "Sheetfile" "servoregulatorsv1.kicad_sch")
+    (property "Sheetfile" "servo_regulator.kicad_sch")
     (property "Sheetname" "")
     (property "ki_description" "Unpolarized capacitor")
@@
     (descr "Capacitor SMD 0805 (2012 Metric), square (rectangular) end terminal, IPC_7351 nominal, (Body size source: IPC-SM-782 page 76, https://www.pcb-3d.com/wordpress/wp-content/uploads/ipc-sm-782a_amendment_1_and_2.pdf, https://docs.google.com/spreadsheets/d/1BsfQQcO9C6DZCsRaXUlFlo91Tg2WpOkGARC1WS5S8t0/edit?usp=sharing), generated with kicad-footprint-generator")
     (tags "capacitor")
-    (property "Sheetfile" "servoregulatorsv1.kicad_sch")
+    (property "Sheetfile" "servo_regulator.kicad_sch")
     (property "Sheetname" "")
     (property "ki_description" "Unpolarized capacitor")
@@
     (descr "Capacitor SMD 0805 (2012 Metric), square (rectangular) end terminal, IPC_7351 nominal, (Body size source: IPC-SM-782 page 76, https://www.pcb-3d.com/wordpress/wp-content/uploads/ipc-sm-782a_amendment_1_and_2.pdf, https://docs.google.com/spreadsheets/d/1BsfQQcO9C6DZCsRaXUlFlo91Tg2WpOkGARC1WS5S8t0/edit?usp=sharing), generated with kicad-footprint-generator")
     (tags "capacitor")
-    (property "Sheetfile" "servoregulatorsv1.kicad_sch")
+    (property "Sheetfile" "servo_regulator.kicad_sch")
     (property "Sheetname" "")
     (property "ki_description" "Unpolarized capacitor")
@@
     (descr "Capacitor SMD 0805 (2012 Metric), square (rectangular) end terminal, IPC_7351 nominal, (Body size source: IPC-SM-782 page 76, https://www.pcb-3d.com/wordpress/wp-content/uploads/ipc-sm-782a_amendment_1_and_2.pdf, https://docs.google.com/spreadsheets/d/1BsfQQcO9C6DZCsRaXUlFlo91Tg2WpOkGARC1WS5S8t0/edit?usp=sharing), generated with kicad-footprint-generator")
     (tags "capacitor")
-    (property "Sheetfile" "servoregulatorsv1.kicad_sch")
+    (property "Sheetfile" "servo_regulator.kicad_sch")
     (property "Sheetname" "")
     (property "ki_description" "Unpolarized capacitor")
@@
     (descr "Inductor, Taiyo Yuden, NR series, Taiyo-Yuden_NR-60xx, 6.0mmx6.0mm")
     (tags "inductor taiyo-yuden nr smd")
-    (property "Sheetfile" "servoregulatorsv1.kicad_sch")
+    (property "Sheetfile" "servo_regulator.kicad_sch")
     (property "Sheetname" "")
     (property "ki_description" "Inductor")
@@
     (descr "Resistor SMD 0603 (1608 Metric), square (rectangular) end terminal, IPC_7351 nominal, (Body size source: IPC-SM-782 page 72, https://www.pcb-3d.com/wordpress/wp-content/uploads/ipc-sm-782a_amendment_1_and_2.pdf), generated with kicad-footprint-generator")
     (tags "resistor")
-    (property "Sheetfile" "servoregulatorsv1.kicad_sch")
+    (property "Sheetfile" "servo_regulator.kicad_sch")
     (property "Sheetname" "")
     (property "ki_description" "Resistor, US symbol")
@@
     (descr "Capacitor SMD 0805 (2012 Metric), square (rectangular) end terminal, IPC_7351 nominal, (Body size source: IPC-SM-782 page 76, https://www.pcb-3d.com/wordpress/wp-content/uploads/ipc-sm-782a_amendment_1_and_2.pdf, https://docs.google.com/spreadsheets/d/1BsfQQcO9C6DZCsRaXUlFlo91Tg2WpOkGARC1WS5S8t0/edit?usp=sharing), generated with kicad-footprint-generator")
     (tags "capacitor")
-    (property "Sheetfile" "servoregulatorsv1.kicad_sch")
+    (property "Sheetfile" "servo_regulator.kicad_sch")
     (property "Sheetname" "")
     (property "ki_description" "Unpolarized capacitor")
@@
     (descr "Capacitor SMD 0805 (2012 Metric), square (rectangular) end terminal, IPC_7351 nominal, (Body size source: IPC-SM-782 page 76, https://www.pcb-3d.com/wordpress/wp-content/uploads/ipc-sm-782a_amendment_1_and_2.pdf, https://docs.google.com/spreadsheets/d/1BsfQQcO9C6DZCsRaXUlFlo91Tg2WpOkGARC1WS5S8t0/edit?usp=sharing), generated with kicad-footprint-generator")
     (tags "capacitor")
-    (property "Sheetfile" "servoregulatorsv1.kicad_sch")
+    (property "Sheetfile" "servo_regulator.kicad_sch")
     (property "Sheetname" "")
     (property "ki_description" "Unpolarized capacitor")
@@
     (descr "Resistor SMD 0603 (1608 Metric), square (rectangular) end terminal, IPC_7351 nominal, (Body size source: IPC-SM-782 page 72, https://www.pcb-3d.com/wordpress/wp-content/uploads/ipc-sm-782a_amendment_1_and_2.pdf), generated with kicad-footprint-generator")
     (tags "resistor")
-    (property "Sheetfile" "servoregulatorsv1.kicad_sch")
+    (property "Sheetfile" "servo_regulator.kicad_sch")
     (property "Sheetname" "")
     (property "ki_description" "Resistor, US symbol")
@@
     (descr "JST EH series connector, B3B-EH-A (http://www.jst-mfg.com/product/pdf/eng/eEH.pdf), generated with kicad-footprint-generator")
     (tags "connector JST EH vertical")
-    (property "Sheetfile" "servoregulatorsv1.kicad_sch")
+    (property "Sheetfile" "servo_regulator.kicad_sch")
     (property "Sheetname" "")
     (property "ki_description" "Generic connector, single row, 01x03, script generated")
@@
     (descr "Resistor SMD 0603 (1608 Metric), square (rectangular) end terminal, IPC_7351 nominal, (Body size source: IPC-SM-782 page 72, https://www.pcb-3d.com/wordpress/wp-content/uploads/ipc-sm-782a_amendment_1_and_2.pdf), generated with kicad-footprint-generator")
     (tags "resistor")
-    (property "Sheetfile" "servoregulatorsv1.kicad_sch")
+    (property "Sheetfile" "servo_regulator.kicad_sch")
     (property "Sheetname" "")
     (property "ki_description" "Resistor, US symbol")
@@
     (descr "JST EH series connector, B3B-EH-A (http://www.jst-mfg.com/product/pdf/eng/eEH.pdf), generated with kicad-footprint-generator")
     (tags "connector JST EH vertical")
-    (property "Sheetfile" "servoregulatorsv1.kicad_sch")
+    (property "Sheetfile" "servo_regulator.kicad_sch")
     (property "Sheetname" "")
     (property "ki_description" "Generic connector, single row, 01x03, script generated")
@@
     (descr "TSOT, 6 Pin (https://www.jedec.org/sites/default/files/docs/MO-193D.pdf variant AA), generated with kicad-footprint-generator ipc_gullwing_generator.py")
     (tags "TSOT TO_SOT_SMD")
-    (property "Sheetfile" "servoregulatorsv1.kicad_sch")
+    (property "Sheetfile" "servo_regulator.kicad_sch")
     (property "Sheetname" "")
     (attr smd)
@@
         (effects (font (size 0.5 0.5) (thickness 0.125)))
     )
-    (fp_text value "~" (at -0.05 2.2 90) (layer "F.Fab")
+    (fp_text value "TPS563208DDCR" (at -0.05 2.2 90) (layer "F.Fab")
         (effects (font (size 1 1) (thickness 0.15)))
     )
@@
     (descr "Capacitor SMD 0805 (2012 Metric), square (rectangular) end terminal, IPC_7351 nominal, (Body size source: IPC-SM-782 page 76, https://www.pcb-3d.com/wordpress/wp-content/uploads/ipc-sm-782a_amendment_1_and_2.pdf, https://docs.google.com/spreadsheets/d/1BsfQQcO9C6DZCsRaXUlFlo91Tg2WpOkGARC1WS5S8t0/edit?usp=sharing), generated with kicad-footprint-generator")
     (tags "capacitor")
-    (property "Sheetfile" "servoregulatorsv1.kicad_sch")
+    (property "Sheetfile" "servo_regulator.kicad_sch")
     (property "Sheetname" "")
     (property "ki_description" "Unpolarized capacitor")
@@
     (descr "SOT, 3 Pin (https://www.jedec.org/system/files/docs/to-236h.pdf variant AB), generated with kicad-footprint-generator ipc_gullwing_generator.py")
     (tags "SOT TO_SOT_SMD")
-    (property "Sheetfile" "servoregulatorsv1.kicad_sch")
+    (property "Sheetfile" "servo_regulator.kicad_sch")
     (property "Sheetname" "")
     (property "ki_description" "0.38A Id, 60V Vds, N-Channel MOSFET, SOT-23")
@@
     (descr "Resistor SMD 0603 (1608 Metric), square (rectangular) end terminal, IPC_7351 nominal, (Body size source: IPC-SM-782 page 72, https://www.pcb-3d.com/wordpress/wp-content/uploads/ipc-sm-782a_amendment_1_and_2.pdf), generated with kicad-footprint-generator")
     (tags "resistor")
-    (property "Sheetfile" "servoregulatorsv1.kicad_sch")
+    (property "Sheetfile" "servo_regulator.kicad_sch")
     (property "Sheetname" "")
     (property "ki_description" "Resistor, US symbol")
@@
         (effects (font (size 1 1) (thickness 0.15)) (justify mirror))
     )
-    (fp_text value "420" (at 0 -1.43) (layer "B.Fab")
+    (fp_text value "430" (at 0 -1.43) (layer "B.Fab")
         (effects (font (size 1 1) (thickness 0.15)) (justify mirror))
     )
@@
     (descr "SOT, 3 Pin (https://www.jedec.org/system/files/docs/to-236h.pdf variant AB), generated with kicad-footprint-generator ipc_gullwing_generator.py")
     (tags "SOT TO_SOT_SMD")
-    (property "Sheetfile" "servoregulatorsv1.kicad_sch")
+    (property "Sheetfile" "servo_regulator.kicad_sch")
     (property "Sheetname" "")
     (property "ki_description" "0.38A Id, 60V Vds, N-Channel MOSFET, SOT-23")
@@
     (descr "Resistor SMD 0603 (1608 Metric), square (rectangular) end terminal, IPC_7351 nominal, (Body size source: IPC-SM-782 page 72, https://www.pcb-3d.com/wordpress/wp-content/uploads/ipc-sm-782a_amendment_1_and_2.pdf), generated with kicad-footprint-generator")
     (tags "resistor")
-    (property "Sheetfile" "servoregulatorsv1.kicad_sch")
+    (property "Sheetfile" "servo_regulator.kicad_sch")
     (property "Sheetname" "")
     (property "ki_description" "Resistor, US symbol")
@@
         (effects (font (size 1 1) (thickness 0.15)) (justify mirror))
     )
-    (fp_text value "420" (at 0 -1.43 90) (layer "B.Fab")
+    (fp_text value "430" (at 0 -1.43 90) (layer "B.Fab")
         (effects (font (size 1 1) (thickness 0.15)) (justify mirror))
     )

Commit message: Adjusted pullup resistors
Parts:
- R4: value 430 -> 10k
- R5: value 430 -> 5.1k
Changed lines of the file:
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@@
         (effects (font (size 1 1) (thickness 0.15)) (justify mirror))
     )
-    (fp_text value "430" (at 0 -1.43) (layer "B.Fab")
+    (fp_text value "5.1k" (at 0 -1.43) (layer "B.Fab")
         (effects (font (size 1 1) (thickness 0.15)) (justify mirror))
     )
@@
         (effects (font (size 1 1) (thickness 0.15)) (justify mirror))
     )
-    (fp_text value "430" (at 0 -1.43 90) (layer "B.Fab")
+    (fp_text value "10k" (at 0 -1.43 90) (layer "B.Fab")
         (effects (font (size 1 1) (thickness 0.15)) (justify mirror))
     )
