File: prop_pitch/prop_pitch.kicad_pcb (KiCad board)
At the start: 2 copper layers, 65 x 22 mm, 54 parts, among them J1 AVR-ISP-6, J2 LOAD1, J3 LOAD2, J4 SERVO1, J6 SERVO2, Q1 MMS8550, U1 ATmega328P-A, U3 HC-05, U4 TPS563208DDCR, U5 AZ1117-5.0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

Commit message: Updated spar sensor to reflect order
Parts:
- Q1: value MMS8550 -> MMBT2907
- R4: value 5k -> 5.1k
- Y1: value Resonator_Small -> 16M
Changed lines of the file:
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@@
   (paper "USLetter")
   (title_block
+    (title "Propellor Pitch and Monitor")
     (date "2023-06-28")
     (rev "1")
+    (company "HPVDT")
   )
   (layers
@@
         (effects (font (size 1 1) (thickness 0.15)))
     )
-    (fp_text value "5k" (at 0 1.43 90) (layer "F.Fab")
+    (fp_text value "5.1k" (at 0 1.43 90) (layer "F.Fab")
         (effects (font (size 1 1) (thickness 0.15)))
     )
@@
         (effects (font (size 1 1) (thickness 0.15)))
     )
-    (fp_text value "MMS8550" (at 0 2.4 90) (layer "F.Fab")
+    (fp_text value "MMBT2907" (at 0 2.4 90) (layer "F.Fab")
         (effects (font (size 1 1) (thickness 0.15)))
     )
@@
         (effects (font (size 1 1) (thickness 0.15)))
     )
-    (fp_text value "Resonator_Small" (at 0 1.8 90) (layer "F.Fab")
+    (fp_text value "16M" (at 0 1.8 90) (layer "F.Fab")
         (effects (font (size 0.2 0.2) (thickness 0.03)))
     )

Commit message: Updated for prop pitch order
Parts:
- Q1: value MMBT2907 -> MMSS8550
- R15, R16, R17: value 330 -> 430
Changed lines of the file:
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@@
         (effects (font (size 1 1) (thickness 0.15)))
     )
-    (fp_text value "MMBT2907" (at 0 2.4 90) (layer "F.Fab")
+    (fp_text value "MMSS8550" (at 0 2.4 90) (layer "F.Fab")
         (effects (font (size 1 1) (thickness 0.15)))
     )
@@
     (property "Sheetfile" "prop_pitch.kicad_sch")
     (property "Sheetname" "")
+    (property "exclude_from_bom" "")
     (property "ki_description" "Generic connector, single row, 01x04, script generated (kicad-library-utils/schlib/autogen/connector/)")
     (property "ki_keywords" "connector")
-    (attr through_hole)
+    (attr through_hole exclude_from_bom)
     (fp_text reference "J2" (at 0 2.33 90) (layer "B.SilkS") hide
         (effects (font (size 1 1) (thickness 0.15)) (justify mirror))
@@
     (property "Sheetfile" "prop_pitch.kicad_sch")
     (property "Sheetname" "")
+    (property "exclude_from_bom" "")
     (property "ki_description" "Generic connector, single row, 01x04, script generated (kicad-library-utils/schlib/autogen/connector/)")
     (property "ki_keywords" "connector")
-    (attr through_hole)
+    (attr through_hole exclude_from_bom)
     (fp_text reference "J3" (at 0 2.33 90) (layer "B.SilkS") hide
         (effects (font (size 1 1) (thickness 0.15)) (justify mirror))
@@
     (property "Sheetfile" "prop_pitch.kicad_sch")
     (property "Sheetname" "")
+    (property "exclude_from_bom" "")
     (property "ki_description" "Multiple-cell battery")
     (property "ki_keywords" "batt voltage-source cell")
-    (attr exclude_from_pos_files)
+    (attr exclude_from_pos_files exclude_from_bom)
     (fp_text reference "BT1" (at 3 2.9 90) (layer "B.SilkS") hide
         (effects (font (size 1 1) (thickness 0.15)) (justify mirror))
@@
         (effects (font (size 1 1) (thickness 0.15)) (justify mirror))
     )
-    (fp_text value "330" (at 0 -1.43 90) (layer "B.Fab")
+    (fp_text value "430" (at 0 -1.43 90) (layer "B.Fab")
         (effects (font (size 1 1) (thickness 0.15)) (justify mirror))
     )
@@
         (effects (font (size 1 1) (thickness 0.15)) (justify mirror))
     )
-    (fp_text value "330" (at 0 -1.43 90) (layer "B.Fab")
+    (fp_text value "430" (at 0 -1.43 90) (layer "B.Fab")
         (effects (font (size 1 1) (thickness 0.15)) (justify mirror))
     )
@@
         (effects (font (size 1 1) (thickness 0.15)) (justify mirror))
     )
-    (fp_text value "330" (at 0 -1.43 90) (layer "B.Fab")
-        (effects (font (size 1 1) (thickness 0.15)) (justify mirror))
-    )
+    (fp_text value "430" (at 0 -1.43 90) (layer "B.Fab")
+        (effects (font (size 1 1) (thickness 0.15)) (justify mirror))
+    )
