File: indicator/indicator.kicad_pcb (KiCad board)
At the start: 2 copper layers, 43.2 x 35.6 mm, 21 parts, among them J1 Conn_01x07_Pin

Commit message: Changed indicator resistor values
Parts:
- R1, R2, R3, R4, R5, R6, R7: value 300 -> 430
