File: main_data/AircraftData.kicad_pcb (KiCad board)
At the start: 2 copper layers, 53.1 x 89.8 mm, 54 parts, among them J1 Orientation, J10 Shaft, J11 Wind Speed, J12 DHT, J13 RPi, J14 USB_C_Receptacle_USB2.0, J15 Control Board, J2 PROG, J3 SPI VIDEO, J4 Barometer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

Commit message: Upgraded STM32
Parts:
- R7: value 5k -> 5.1k
- U1: value STM32F103C8Tx -> STM32F103CBTx
- Y1: value 8MHz -> 8M
Changed lines of the file:
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@@
     (property "Sheetfile" "AircraftData.kicad_sch")
     (property "Sheetname" "")
+    (property "exclude_from_bom" "")
     (property "ki_description" "Mounting Hole without connection")
     (property "ki_keywords" "mounting hole")
-    (attr exclude_from_pos_files)
+    (attr exclude_from_pos_files exclude_from_bom)
     (fp_text reference "H2" (at 0 -4.2) (layer "F.SilkS") hide
         (effects (font (size 1 1) (thickness 0.15)))
@@
     (property "Sheetfile" "AircraftData.kicad_sch")
     (property "Sheetname" "")
+    (property "exclude_from_bom" "")
     (property "ki_description" "Mounting Hole without connection")
     (property "ki_keywords" "mounting hole")
-    (attr exclude_from_pos_files)
+    (attr exclude_from_pos_files exclude_from_bom)
     (fp_text reference "H1" (at 0 -4.2) (layer "F.SilkS") hide
         (effects (font (size 1 1) (thickness 0.15)))
@@
         (effects (font (size 1 1) (thickness 0.15)))
     )
-    (fp_text value "8MHz" (at 0 1.8 90) (layer "F.Fab")
+    (fp_text value "8M" (at 0 1.8 90) (layer "F.Fab")
         (effects (font (size 0.2 0.2) (thickness 0.03)))
     )
@@
         (effects (font (size 1 1) (thickness 0.15)))
     )
-    (fp_text value "5k" (at 0 1.43) (layer "F.Fab")
+    (fp_text value "5.1k" (at 0 1.43) (layer "F.Fab")
         (effects (font (size 1 1) (thickness 0.15)))
     )
@@
     (property "Sheetfile" "AircraftData.kicad_sch")
     (property "Sheetname" "")
+    (property "exclude_from_bom" "")
     (property "ki_description" "Jumper, 3-pole, both open")
     (property "ki_keywords" "Jumper SPDT")
-    (attr through_hole)
+    (attr through_hole exclude_from_bom)
     (fp_text reference "JP1" (at 0 -2.33 90) (layer "F.SilkS") hide
         (effects (font (size 1 1) (thickness 0.15)))
@@
     (property "Sheetfile" "AircraftData.kicad_sch")
     (property "Sheetname" "")
-    (property "ki_description" "STMicroelectronics Arm Cortex-M3 MCU, 64KB flash, 20KB RAM, 72 MHz, 2.0-3.6V, 37 GPIO, LQFP48")
+    (property "ki_description" "STMicroelectronics Arm Cortex-M3 MCU, 128KB flash, 20KB RAM, 72 MHz, 2.0-3.6V, 37 GPIO, LQFP48")
     (property "ki_keywords" "Arm Cortex-M3 STM32F1 STM32F103")
     (attr smd)
@@
         (effects (font (size 1 1) (thickness 0.15)))
     )
-    (fp_text value "STM32F103C8Tx" (at 0 5.85) (layer "F.Fab")
+    (fp_text value "STM32F103CBTx" (at 0 5.85) (layer "F.Fab")
         (effects (font (size 1 1) (thickness 0.15)))
     )
@@
     (property "Sheetfile" "AircraftData.kicad_sch")
     (property "Sheetname" "")
+    (property "exclude_from_bom" "")
     (property "ki_description" "Mounting Hole without connection")
     (property "ki_keywords" "mounting hole")
-    (attr exclude_from_pos_files)
+    (attr exclude_from_pos_files exclude_from_bom)
     (fp_text reference "H3" (at 0 -4.2) (layer "F.SilkS") hide
         (effects (font (size 1 1) (thickness 0.15)))
