File: power_monitor/power_monitor_EunGuRevision.kicad_sch (KiCad schematic)
At the start: 25 parts, among them J1 AVR-ISP-6, J2 Conn_01x06_Female, J3 Conn_01x04_Socket, J4 BATT, J5 VEH, U2 ACS712ELCTR-20A, U3 TS2940CW50, X1 ATmega328-A, Y1 16M

Commit message: Finished schematic
Updated with new ADC and added voltage regulator
Parts:
- added C11: 0.1uF, Capacitor_SMD:C_0603_1608Metric, symbol Device:C
- added C12, C13: 10uF, Capacitor_SMD:C_0805_2012Metric, symbol Device:C
- added C14: 22uF, Capacitor_SMD:C_0805_2012Metric, symbol Device:C
- added R2: 10k, Resistor_SMD:R_0603_1608Metric, symbol Device:R
- added U4: AZ1117-3.3, Package_TO_SOT_SMD:SOT-223-3_TabPin2, symbol Regulator_Linear:AZ1117-3.3
- C10, C4: footprint Capacitor_SMD:C_0603_1608Metric -> Capacitor_SMD:C_0805_2012Metric
- MCP1: footprint (none) -> ADC Pretty:QFN-12_EP_2x2_Pitch0.4mm
- R4: value 10k -> 30k
- R5: value 20k -> 10k
- Y1: value 16M -> 8M
Connections:
- net BATT_DIVIDED 10V to 3.3V is gone; now on net BATT_DIVIDED: R4.2, R5.1
- net +5V: no longer C1.1, C2.1, X1.18 (AVCC), X1.4 (VCC), X1.6 (VCC)
- net GND: now also C10.2, C9.2, MCP1.2 (REFIN-), C11.2, C12.2, C13.2, C14.2, U4.1 (GND); no longer C3.1, C4.1, MCP1.3 (REFIN+)
- net MISO: now also MCP1.9 (SDO)
- net MOSI: now also MCP1.8 (SDI)
- net RESET: now also J1.5 (~{RST})
- net SCK: now also MCP1.7 (SCK)
- net SS: no longer J1.5 (~{RST})
- net +3V3: now reaches C10.1, C9.1
- net +3V3: now also C1.1, C2.1, MCP1.11 (DVDD), MCP1.12 (AVDD), X1.18 (AVCC), X1.4 (VCC), X1.6 (VCC), C11.1, C12.1, C13.1, C14.1, R2.2, U4.2 (VO), U4.3 (VI)
- net CS: now reaches X1.12 (PB0)
- net CS: now also MCP1.6 (CS), R2.1
- net BATT_DIVIDED: now reaches MCP1.4 (CH1)
- new net: C3.1, C4.1, MCP1.3 (REFIN+)
- no-connect marks 17 -> 16
Other:
- moved on the sheet: C10, C3, C4, C9
