File: power_monitor/power_monitor_EunGuRevision.kicad_pcb (KiCad board)
At the start: 2 copper layers, 31 parts, among them J1 AVR-ISP-6, J2 Conn_01x06_Female, J3 Conn_01x04_Socket, J4 BATT, J5 VEH, U2 ACS712ELCTR-20A, U3 TS2940CW50, U4 AZ1117-3.3, X1 ATmega328-A, Y1 8M

Commit message: PCB Arrangement
uh Savo how do I do this. I just grouped everything that needed to be together but I didn't fully finish. Also I'll send it over discord in case this isn't the right one
Parts:
- moved R2 69.5 mm to (82.9, 102.2)
- moved J3 66.6 mm to (92.7, 133.3)
- moved X1 63.2 mm to (96.5, 99.0), turned to 180 degrees
- moved C13 63.1 mm to (85.2, 52.6)
- moved C14 61.8 mm to (85.0, 57.5)
- moved C7 59.1 mm to (118.2, 121.9), turned to 90 degrees
- moved C2 58.3 mm to (87.6, 99.8)
- moved J1 57.8 mm to (84.7, 89.1)
- moved C1 57.7 mm to (87.4, 95.8)
- moved U4 56.7 mm to (92.2, 55.3)
- moved R4 54.7 mm to (93.2, 89.7)
- moved R5 53.2 mm to (93.2, 85.2), turned to 180 degrees
- moved Y1 51.3 mm to (103.8, 97.6), turned to -90 degrees
- moved MCP1 42.9 mm to (97.6, 87.2), turned to -90 degrees
- moved C3 42.3 mm to (96.8, 82.8), turned to 90 degrees
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