File: power_monitor/power_monitor.kicad_pcb (KiCad board)
At the start: 2 copper layers, 40 x 50 mm, 35 parts, among them J1 AVR-ISP-6, J2 Conn_01x06_Female, J3 Conn_01x04_Socket, J4 BATT, J5 VEH, U1 ATmega328-A, U2 ACS712ELCTR-20A, U4 AZ1117-3.3, U5 TS2940CW50, Y1 8M

Commit message: Bro where is my last update
Added a name and some author stuff
Other:
- board text added: "Shelly the Power Monitor By Eun Gu Special contributions by Savo, Kassie, and Melani"
Changed lines of the file:
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@@
         (effects (font (size 1 1) (thickness 0.15)))
     )
-    (fp_text value "VEH" (at 3.7 5.25 90) (layer "F.Fab")
+    (fp_text value "VEH" (at 3.9 5.3 90) (layer "F.Fab")
         (effects (font (size 1 1) (thickness 0.15)))
     )
@@
         (effects (font (size 1 1) (thickness 0.15)))
     )
-    (fp_text value "BATT" (at 3.6 5.4 90) (layer "F.Fab")
+    (fp_text value "BATT" (at 10.4 -6.5 180) (layer "F.Fab")
         (effects (font (size 1 1) (thickness 0.15)))
     )
@@
   (gr_rect locked (start 128.25 74) (end 168.25 124)
     (stroke (width 0.2) (type default)) (fill none) (layer "Edge.Cuts"))
+  (gr_text "Shelly the Power Monitor\nBy Eun Gu\nSpecial contributions by Savo, Kassie, and Melani" (at 167.4 122.8) (layer "B.SilkS")
+    (effects (font (size 1 1) (thickness 0.1)) (justify left bottom mirror))
+  )
   (segment (start 157.9 101.3) (end 158.025 101.425) (width 0.2) (layer "F.Cu") (net 1))
   (segment (start 153.875 101.15) (end 152.05 101.15) (width 0.2) (layer "F.Cu") (net 1))

Commit message: More pretty edits
Now that I know what the layers really are it makes a lot more sense
Other:
- board text added: "BATT"
- board text added: "Shelly the Power Monitor By Eun Gu Special contributions: Savo, Kassie, Melani"
- board text added: "VEH"
- board text removed: "Shelly the Power Monitor By Eun Gu Special contributions by Savo, Kassie, and Melani"
Changed lines of the file:
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@@
     (property "ki_keywords" "connector")
     (attr through_hole)
-    (fp_text reference "J2" (at 0 -2.33 90) (layer "F.SilkS")
+    (fp_text reference "J2" (at -0.6 -2.6 180) (layer "F.SilkS")
         (effects (font (size 1 1) (thickness 0.15)))
     )
@@
     (property "ki_keywords" "cap capacitor")
     (attr smd)
-    (fp_text reference "C1" (at 2.45 0) (layer "F.SilkS")
+    (fp_text reference "C1" (at 2.3 0.1) (layer "F.SilkS")
         (effects (font (size 1 1) (thickness 0.15)))
     )
@@
     (property "ki_keywords" "hall effect current monitor sensor isolated")
     (attr smd)
-    (fp_text reference "U2" (at 0 -3.4 90) (layer "F.SilkS")
+    (fp_text reference "U2" (at 0 3.5 90) (layer "F.SilkS")
         (effects (font (size 1 1) (thickness 0.15)))
     )
@@
     (property "ki_keywords" "cap capacitor")
     (attr smd)
-    (fp_text reference "C10" (at 0 -1.68 90) (layer "F.SilkS")
+    (fp_text reference "C10" (at 0.1 -1.7 -90) (layer "F.SilkS")
         (effects (font (size 1 1) (thickness 0.15)))
     )
@@
     (property "ki_keywords" "AVR ISP Connector")
     (attr smd)
-    (fp_text reference "J1" (at 2.425 5.25) (layer "F.SilkS")
+    (fp_text reference "J1" (at 0.075 4.8) (layer "F.SilkS")
         (effects (font (size 1 1) (thickness 0.15)))
     )
@@
     (property "ki_keywords" "connector")
     (attr through_hole)
-    (fp_text reference "J5" (at -4.15 -3.95 180) (layer "F.SilkS")
-        (effects (font (size 1 1) (thickness 0.15)))
-    )
-    (fp_text value "VEH" (at 3.9 5.3 90) (layer "F.Fab")
+    (fp_text reference "J5" (at 12.3 -3.1 180) (layer "F.SilkS")
+        (effects (font (size 1 1) (thickness 0.15)))
+    )
+    (fp_text value "VEH" (at 3.9 5.3 90) (layer "F.Fab") hide
         (effects (font (size 1 1) (thickness 0.15)))
     )
@@
     (property "ki_keywords" "Fixed Voltage Regulator 1A Positive LDO")
     (attr smd)
-    (fp_text reference "U4" (at 0 4.45) (layer "F.SilkS")
+    (fp_text reference "U4" (at 3.15 3.1) (layer "F.SilkS")
         (effects (font (size 1 1) (thickness 0.15)))
     )
@@
     (property "ki_keywords" "cap capacitor")
     (attr smd)
-    (fp_text reference "C4" (at 2.648 0.069) (layer "F.SilkS")
+    (fp_text reference "C4" (at 2.448 0.069) (layer "F.SilkS")
         (effects (font (size 1 1) (thickness 0.15)))
     )
@@
     (property "ki_keywords" "solder jumper SPST")
     (attr exclude_from_pos_files)
-    (fp_text reference "JP1" (at 2.5 0 -180) (layer "F.SilkS")
+    (fp_text reference "JP1" (at -2.3 0 -180) (layer "F.SilkS")
         (effects (font (size 1 1) (thickness 0.15)))
     )
@@
     (property "ki_keywords" "R res resistor")
     (attr smd)
-    (fp_text reference "R4" (at 2.625 -0.1 90) (layer "F.SilkS")
+    (fp_text reference "R4" (at 2.425 -0.1 90) (layer "F.SilkS")
         (effects (font (size 1 1) (thickness 0.15)))
     )
@@
     (property "ki_keywords" "cap capacitor")
     (attr smd)
-    (fp_text reference "C12" (at -1.3 -2.7 90) (layer "F.SilkS")
+    (fp_text reference "C12" (at 3.1 -0.3 180) (layer "F.SilkS")
         (effects (font (size 1 1) (thickness 0.15)))
     )
@@
     (property "ki_keywords" "R res resistor")
     (attr smd)
-    (fp_text reference "R3" (at -2.575 -0.1 90) (layer "F.SilkS")
+    (fp_text reference "R3" (at 0.025 1.9 -180) (layer "F.SilkS")
         (effects (font (size 1 1) (thickness 0.15)))
     )
@@
     (property "ki_keywords" "R res resistor")
     (attr smd)
-    (fp_text reference "R1" (at 0 -1.43 90) (layer "F.SilkS")
+    (fp_text reference "R1" (at -1.025 1.4 90) (layer "F.SilkS")
         (effects (font (size 1 1) (thickness 0.15)))
     )
@@
     (property "ki_keywords" "connector")
     (attr through_hole)
-    (fp_text reference "J3" (at 2.55 -4.5 90) (layer "F.SilkS")
+    (fp_text reference "J3" (at 11.35 -0.1 -180) (layer "F.SilkS")
         (effects (font (size 1 1) (thickness 0.15)))
     )
@@
     (property "ki_keywords" "cap capacitor")
     (attr smd)
-    (fp_text reference "C13" (at 1 -2.53 90) (layer "F.SilkS")
+    (fp_text reference "C13" (at 0.9 -2.5 180) (layer "F.SilkS")
         (effects (font (size 1 1) (thickness 0.15)))
     )
@@
     (property "ki_keywords" "ceramic resonator")
     (attr smd)
-    (fp_text reference "Y1" (at 0 -2) (layer "F.SilkS")
+    (fp_text reference "Y1" (at -3.1 -0.1) (layer "F.SilkS")
         (effects (font (size 1 1) (thickness 0.15)))
     )
@@
     (property "ki_keywords" "connector")
     (attr through_hole)
-    (fp_text reference "J4" (at -5.6 0.1 180) (layer "F.SilkS")
-        (effects (font (size 1 1) (thickness 0.15)))
-    )
-    (fp_text value "BATT" (at 10.4 -6.5 180) (layer "F.Fab")
+    (fp_text reference "J4" (at 12.6 2.1 180) (layer "F.SilkS")
+        (effects (font (size 1 1) (thickness 0.15)))
+    )
+    (fp_text value "BATT" (at 10.4 -6.5 180) (layer "F.Fab") hide
         (effects (font (size 1 1) (thickness 0.15)))
     )
@@
     (property "ki_keywords" "cap capacitor")
     (attr smd)
-    (fp_text reference "C3" (at 0 -1.6) (layer "F.SilkS")
+    (fp_text reference "C3" (at 0 -1.4) (layer "F.SilkS")
         (effects (font (size 1 1) (thickness 0.15)))
     )
@@
     (property "ki_keywords" "AVR 8bit Microcontroller MegaAVR")
     (attr smd)
-    (fp_text reference "U1" (at 0 -6.05 90) (layer "F.SilkS")
+    (fp_text reference "U1" (at 4.5 -4.25 180) (layer "F.SilkS")
         (effects (font (size 1 1) (thickness 0.15)))
     )
@@
     (property "ki_keywords" "cap capacitor")
     (attr smd)
-    (fp_text reference "C7" (at 0 -1.43 90) (layer "F.SilkS")
+    (fp_text reference "C7" (at 2.6 -0.175 90) (layer "F.SilkS")
         (effects (font (size 1 1) (thickness 0.15)))
     )
@@
     (property "ki_keywords" "cap capacitor")
     (attr smd)
-    (fp_text reference "C5" (at 2.15 -0.025 -180) (layer "F.SilkS")
+    (fp_text reference "C5" (at 2.55 -0.225 -90) (layer "F.SilkS")
         (effects (font (size 1 1) (thickness 0.15)))
     )
@@
     (property "ki_description" "5V Linear regulator")
     (attr smd)
-    (fp_text reference "U5" (at 0 -4.5) (layer "F.SilkS")
+    (fp_text reference "U5" (at 3.15 -3.15) (layer "F.SilkS")
         (effects (font (size 1 1) (thickness 0.15)))
     )
@@
     (property "ki_keywords" "cap capacitor")
     (attr smd)
-    (fp_text reference "C2" (at 2.7 -0.05) (layer "F.SilkS")
+    (fp_text reference "C2" (at 2.3 0.35) (layer "F.SilkS")
         (effects (font (size 1 1) (thickness 0.15)))
     )
@@
   (gr_rect locked (start 128.25 74) (end 168.25 124)
     (stroke (width 0.2) (type default)) (fill none) (layer "Edge.Cuts"))
-  (gr_text "Shelly the Power Monitor\nBy Eun Gu\nSpecial contributions by Savo, Kassie, and Melani" (at 167.4 122.8) (layer "B.SilkS")
+  (gr_text "Shelly the Power Monitor\nBy Eun Gu\nSpecial contributions: Savo, Kassie, Melani" (at 167.2 115.6) (layer "B.SilkS")
     (effects (font (size 1 1) (thickness 0.1)) (justify left bottom mirror))
   )
+  (gr_text "BATT" (at 154.4 85.2) (layer "F.SilkS" knockout)
+    (effects (font (size 1 1) (thickness 0.1)) (justify left bottom))
+  )
+  (gr_text "VEH\n" (at 138.4 85.4) (layer "F.SilkS" knockout)
+    (effects (font (size 1 1) (thickness 0.1)) (justify left bottom))
+  )
   (segment (start 157.9 101.3) (end 158.025 101.425) (width 0.2) (layer "F.Cu") (net 1))
