File: power_monitor/power_monitor.kicad_pcb (KiCad board)
At the start: 2 copper layers, 40 x 50 mm, 35 parts, among them J1 AVR-ISP-6, J2 Conn_01x06_Female, J3 Conn_01x04_Socket, J4 BATT, J5 VEH, U1 ATmega328-A, U2 ACS712ELCTR-20A, U4 AZ1117-3.3, U5 TS2940CW50, Y1 8M

Commit message: pls let this end
label. bigger.
Parts:
- moved R3 0.53 mm to (157.2, 88.0)
- moved R4 0.53 mm to (157.2, 91.0)
Routing:
- net /BATT_DIVIDED: track 13.4 -> 14.0 mm
Other:
- board text added: "BAT"
- board text removed: "BATT"
Changed lines of the file:
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@@
     (property "ki_keywords" "hall effect current monitor sensor isolated")
     (attr smd)
-    (fp_text reference "U2" (at 0 3.5 90) (layer "F.SilkS")
+    (fp_text reference "U2" (at -4.6 0.1 -180) (layer "F.SilkS")
         (effects (font (size 1 1) (thickness 0.15)))
     )
@@
     (property "ki_keywords" "cap capacitor")
     (attr smd)
-    (fp_text reference "C10" (at 0.1 -1.7 -90) (layer "F.SilkS")
+    (fp_text reference "C10" (at 0.9 -1.9 -90) (layer "F.SilkS")
         (effects (font (size 1 1) (thickness 0.15)))
     )
@@
     (property "ki_keywords" "AVR ISP Connector")
     (attr smd)
-    (fp_text reference "J1" (at 0.075 4.8) (layer "F.SilkS")
+    (fp_text reference "J1" (at 6.875 1.2) (layer "F.SilkS")
         (effects (font (size 1 1) (thickness 0.15)))
     )
@@
   )
   (footprint "Resistor_SMD:R_0603_1608Metric" (layer "F.Cu")
-    (at 156.7 91.175 -90)
+    (at 157.2 91 -90)
     (descr "Resistor SMD 0603 (1608 Metric), square (rectangular) end terminal, IPC_7351 nominal, (Body size source: IPC-SM-782 page 72, https://www.pcb-3d.com/wordpress/wp-content/uploads/ipc-sm-782a_amendment_1_and_2.pdf), generated with kicad-footprint-generator")
     (tags "resistor")
@@
     (property "ki_keywords" "R res resistor")
     (attr smd)
-    (fp_text reference "R4" (at 2.425 -0.1 90) (layer "F.SilkS")
+    (fp_text reference "R4" (at 2.6 -0.2 90) (layer "F.SilkS")
         (effects (font (size 1 1) (thickness 0.15)))
     )
@@
   )
   (footprint "Resistor_SMD:R_0603_1608Metric" (layer "F.Cu")
-    (at 156.7 88.175 -90)
+    (at 157.2 88 -90)
     (descr "Resistor SMD 0603 (1608 Metric), square (rectangular) end terminal, IPC_7351 nominal, (Body size source: IPC-SM-782 page 72, https://www.pcb-3d.com/wordpress/wp-content/uploads/ipc-sm-782a_amendment_1_and_2.pdf), generated with kicad-footprint-generator")
     (tags "resistor")
@@
     (property "ki_keywords" "R res resistor")
     (attr smd)
-    (fp_text reference "R3" (at 0.025 1.9 -180) (layer "F.SilkS")
+    (fp_text reference "R3" (at -2.6 0 -90) (layer "F.SilkS")
         (effects (font (size 1 1) (thickness 0.15)))
     )
@@
     (property "ki_keywords" "cap capacitor")
     (attr smd)
-    (fp_text reference "C8" (at -2.5 -0.2 90) (layer "F.SilkS")
+    (fp_text reference "C8" (at -2.9 0 90) (layer "F.SilkS")
         (effects (font (size 1 1) (thickness 0.15)))
     )
@@
     (effects (font (size 1 1) (thickness 0.1)) (justify left bottom mirror))
   )
-  (gr_text "BATT" (at 152 84.8) (layer "F.SilkS" knockout)
-    (effects (font (size 1.65 1.65) (thickness 0.1)) (justify left bottom))
-  )
-  (gr_text "VEH\n" (at 139.2 84.8) (layer "F.SilkS" knockout)
-    (effects (font (size 1.65 1.65) (thickness 0.1)) (justify left bottom))
+  (gr_text "BAT" (at 155.4 89.2 90) (layer "F.SilkS" knockout)
+    (effects (font (size 2 2) (thickness 0.4) bold) (justify left bottom))
+  )
+  (gr_text "VEH\n" (at 144 93 90) (layer "F.SilkS" knockout)
+    (effects (font (size 3 3) (thickness 0.6) bold) (justify left bottom))
   )
   (segment (start 157.9 101.3) (end 158.025 101.425) (width 0.2) (layer "F.Cu") (net 1))
@@
   (segment (start 134.25 109.75) (end 134.9 109.1) (width 0.2) (layer "F.Cu") (net 15))
   (segment (start 134.9 109.1) (end 143.2 109.1) (width 0.2) (layer "F.Cu") (net 15))
+  (segment (start 151.577 92.998462) (end 153.7 95.121462) (width 0.2) (layer "F.Cu") (net 17))
   (segment (start 153.7 95.121462) (end 153.7 97.45) (width 0.2) (layer "F.Cu") (net 17))
+  (segment (start 152.290538 91.35) (end 151.577 92.063538) (width 0.2) (layer "F.Cu") (net 17))
+  (segment (start 156.025 91.35) (end 152.290538 91.35) (width 0.2) (layer "F.Cu") (net 17))
+  (segment (start 157.2 88.825) (end 157.2 90.175) (width 0.2) (layer "F.Cu") (net 17))
   (segment (start 151.577 92.063538) (end 151.577 92.998462) (width 0.2) (layer "F.Cu") (net 17))
-  (segment (start 151.577 92.998462) (end 153.7 95.121462) (width 0.2) (layer "F.Cu") (net 17))
-  (segment (start 156.7 90.35) (end 155.7 91.35) (width 0.2) (layer "F.Cu") (net 17))
-  (segment (start 156.7 89) (end 156.7 90.35) (width 0.2) (layer "F.Cu") (net 17))
-  (segment (start 155.7 91.35) (end 152.290538 91.35) (width 0.2) (layer "F.Cu") (net 17))
-  (segment (start 152.290538 91.35) (end 151.577 92.063538) (width 0.2) (layer "F.Cu") (net 17))
+  (segment (start 157.2 90.175) (end 156.025 91.35) (width 0.2) (layer "F.Cu") (net 17))
   (segment (start 153.3 95.3) (end 153.3 97.45) (width 0.2) (layer "F.Cu") (net 18))
   (segment (start 149.335 93.335) (end 150.25 94.25) (width 0.2) (layer "F.Cu") (net 18))

Commit message: Small edits
Moved around the text on back and moved the trace by the mounting hole.
Routing:
- net +5V: track 83.1 -> 85.2 mm
Changed lines of the file:
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@@
     (property "ki_keywords" "cap capacitor")
     (attr smd)
-    (fp_text reference "C12" (at 3.1 -0.3 180) (layer "F.SilkS")
+    (fp_text reference "C12" (at 3.3 -0.5 180) (layer "F.SilkS")
         (effects (font (size 1 1) (thickness 0.15)))
     )
@@
     (property "ki_keywords" "cap capacitor")
     (attr smd)
-    (fp_text reference "C13" (at 0.9 -2.5 180) (layer "F.SilkS")
+    (fp_text reference "C13" (at 1.9 -2.5 180) (layer "F.SilkS")
         (effects (font (size 1 1) (thickness 0.15)))
     )
@@
   (gr_rect locked (start 128.25 74) (end 168.25 124)
     (stroke (width 0.2) (type default)) (fill none) (layer "Edge.Cuts"))
-  (gr_text "Shelly the Power Monitor\nBy Eun Gu\nSpecial contributions: Savo, Kassie, Melani" (at 167.2 115.6) (layer "B.SilkS")
+  (gr_text "Shelly the Power Monitor\nBy Eun Gu\nSpecial contributions: Savo, \nKassie, Melani" (at 158.8 122.6) (layer "B.SilkS")
     (effects (font (size 1 1) (thickness 0.1)) (justify left bottom mirror))
   )
@@
   (via (at 147.4 77.5) (size 0.6) (drill 0.3) (layers "F.Cu" "B.Cu") (net 1))
   (via (at 141.1 78.3) (size 0.6) (drill 0.3) (layers "F.Cu" "B.Cu") (net 1))
+  (segment (start 159.2 75.75) (end 159.95 75) (width 0.2) (layer "F.Cu") (net 3))
   (segment (start 156.7 75.95) (end 146.25 75.95) (width 0.2) (layer "F.Cu") (net 3))
+  (segment (start 167.6 75) (end 167.6 104.8) (width 0.2) (layer "F.Cu") (net 3))
   (segment (start 150.605 90.475) (end 150.777 90.647) (width 0.2) (layer "F.Cu") (net 3))
   (segment (start 141.6 80.6) (end 141.1 80.6) (width 0.2) (layer "F.Cu") (net 3))
   (segment (start 138.85 80.9) (end 139.15 80.6) (width 0.2) (layer "F.Cu") (net 3))
+  (segment (start 159.95 75) (end 167.6 75) (width 0.2) (layer "F.Cu") (net 3))
   (segment (start 156.7 75.95) (end 159 75.95) (width 0.2) (layer "F.Cu") (net 3))
-  (segment (start 166.2 78.242284) (end 166.2 106.2) (width 0.2) (layer "F.Cu") (net 3))
+  (segment (start 167.6 104.8) (end 166.2 106.2) (width 0.2) (layer "F.Cu") (net 3))
   (segment (start 159 75.95) (end 159.2 75.75) (width 0.2) (layer "F.Cu") (net 3))
   (segment (start 139.15 80.6) (end 141.1 80.6) (width 0.2) (layer "F.Cu") (net 3))
   (segment (start 156.7 75.95) (end 156.7 76.950498) (width 0.2) (layer "F.Cu") (net 3))
   (segment (start 151.75 90.75) (end 150.88 90.75) (width 0.2) (layer "F.Cu") (net 3))
-  (segment (start 163.907716 75.95) (end 166.2 78.242284) (width 0.2) (layer "F.Cu") (net 3))
   (segment (start 156.7 76.950498) (end 156.75 77.000498) (width 0.2) (layer "F.Cu") (net 3))
-  (segment (start 156.7 75.95) (end 163.907716 75.95) (width 0.2) (layer "F.Cu") (net 3))
   (segment (start 146.25 75.95) (end 141.6 80.6) (width 0.2) (layer "F.Cu") (net 3))
   (segment (start 150.777 90.647) (end 150.777 92.531) (width 0.2) (layer "F.Cu") (net 3))
