File: power_monitor/power_monitor.kicad_sch (KiCad schematic)
At the start: 24 parts, among them J1 BATT, J2 VEH, J3 AVR-ISP-6, J4 Conn_01x06_Female, U1 ACS712ELCTR-20A, U2 MCP3426A0T-E/SN, U3 TS2940CW50, X1 ATmega328-A, Y1 16 MHz Crystal

Commit message: Touched up schematic
Parts:
- removed C1, C2: 22 pF, symbol Device:C
- removed Y1: 16 MHz Crystal, symbol Device:Crystal
- added C4: 100 nF, symbol Device:C
- added J3: Conn_01x04_Socket, Connector_JST:JST_XA_B04B-XASK-1_1x04_P2.50mm_Vertical, symbol Connector:Conn_01x04_Socket
- added JP1: Power Connect, Jumper:SolderJumper-2_P1.3mm_Open_Pad1.0x1.5mm, symbol Jumper:SolderJumper_2_Open
- added Y1: 16M, Crystal:Resonator_SMD_Murata_CSTxExxV-3Pin_3.0x1.1mm, symbol Device:Resonator_Small
- C6: renamed from C5; value 0.1 uF -> 100 nF
- J2: renamed from J4; footprint (none) -> Connector_PinHeader_2.54mm:PinHeader_1x06_P2.54mm_Vertical
- S1: value SW_RST -> RST
- renumbered C9 to C1, C8 to C2, C7 to C3, C6 to C5, C3 to C7, C4 to C8, J3 to J1, J1 to J4, J2 to J5, R_RST1 to R1, R_SDA1 to R2, R_SCL1 to R3, R1 to R4, R2 to R5, U2 to U1, U1 to U2
Connections:
- net GND: now also C4.2, J3.1 (Pin_1), Y1.2
- net SCL: now also J3.4 (Pin_4)
- net SDA: now also J3.3 (Pin_3)
- net at X1.7 (XTAL1/PB6): now also Y1.3
- net at X1.8 (XTAL2/PB7): now also Y1.1
- net BATT_DIVIDED: now reaches R4.2, R5.1, U1.1 (CH1+)
- net CURRENT: now reaches U1.7 (CH2+), U2.7 (VIOUT)
- net 5V_reg renamed +5V
- net +5V: now also C4.1, JP1.1 (A)
- net BATT renamed +BATT
- new net: J3.2 (Pin_2), JP1.2 (B)
Other:
- moved on the sheet: C1, C2, C5, C6, C7, C8, J1, J2, U3

Commit message: Set footprints, touched up regulator symbol
Parts:
- C1, C2, C3, C4, C5, C6, C7: footprint (none) -> Capacitor_SMD:C_0603_1608Metric
- C8: footprint (none) -> Capacitor_SMD:C_0805_2012Metric
- J1: footprint (none) -> Connector_PinHeader_2.54mm:PinHeader_2x03_P2.54mm_Vertical_SMD
- R1, R2, R3, R4, R5: footprint (none) -> Resistor_SMD:R_0603_1608Metric
- S1: footprint (none) -> Button_Switch_SMD:SW_SPST_SKQG_WithStem
- U1: footprint (none) -> Package_SO:SOIC-8_3.9x4.9mm_P1.27mm
- U3: footprint (none) -> Package_TO_SOT_SMD:SOT-223-3_TabPin2; symbol New_Library:TS2940CW50 -> TS2940CW50:TS2940CW50
Changed lines of the file:
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@@
     )
   )
-  (symbol (lib_id "New_Library:TS2940CW50") (at 237.49 143.51 0) (unit 1)
+  (symbol (lib_id "TS2940CW50:TS2940CW50") (at 237.49 143.51 0) (unit 1)
     (in_bom yes) (on_board yes) (dnp no) (fields_autoplaced)
     (property "Reference" "U3" (at 237.49 130.81 0)
@@
       (effects (font (size 1.27 1.27)))
     )
-    (property "Footprint" "" (at 237.49 143.51 0)
-      (effects (font (size 1.27 1.27)) hide)
-    )
-    (property "Datasheet" "" (at 237.49 143.51 0)
+    (property "Footprint" "Package_TO_SOT_SMD:SOT-223-3_TabPin2" (at 237.49 149.86 0)
+      (effects (font (size 1.27 1.27)) hide)
+    )
+    (property "Datasheet" "https://www.taiwansemi.com/assets/uploads/datasheet/TS2940_D15.pdf" (at 237.49 152.4 0)
       (effects (font (size 1.27 1.27)) hide)
     )
@@
       (effects (font (size 1.27 1.27)) (justify right))
     )
-    (property "Footprint" "" (at 115.062 58.42 90)
+    (property "Footprint" "Resistor_SMD:R_0603_1608Metric" (at 115.062 58.42 90)
       (effects (font (size 1.27 1.27)) hide)
     )
@@
       (effects (font (size 1.27 1.27)) (justify left))
     )
-    (property "Footprint" "" (at 39.0652 38.1 0)
+    (property "Footprint" "Capacitor_SMD:C_0603_1608Metric" (at 39.0652 38.1 0)
       (effects (font (size 1.27 1.27)) hide)
     )
@@
       (effects (font (size 1.27 1.27)) (justify left))
     )
-    (property "Footprint" "" (at 221.9452 148.59 0)
+    (property "Footprint" "Capacitor_SMD:C_0603_1608Metric" (at 221.9452 148.59 0)
       (effects (font (size 1.27 1.27)) hide)
     )
@@
       (effects (font (size 1.27 1.27)) (justify left))
     )
-    (property "Footprint" "" (at 166.0652 124.46 0)
+    (property "Footprint" "Capacitor_SMD:C_0603_1608Metric" (at 166.0652 124.46 0)
       (effects (font (size 1.27 1.27)) hide)
     )
@@
       (effects (font (size 1.27 1.27)) (justify left))
     )
-    (property "Footprint" "" (at 28.702 73.66 90)
+    (property "Footprint" "Resistor_SMD:R_0603_1608Metric" (at 28.702 73.66 90)
       (effects (font (size 1.27 1.27)) hide)
     )
@@
       (effects (font (size 1.27 1.27)) (justify left))
     )
-    (property "Footprint" "" (at 183.642 64.77 90)
+    (property "Footprint" "Resistor_SMD:R_0603_1608Metric" (at 183.642 64.77 90)
       (effects (font (size 1.27 1.27)) hide)
     )
@@
       (effects (font (size 1.27 1.27)) (justify left))
     )
-    (property "Footprint" "" (at 183.642 53.34 90)
+    (property "Footprint" "Resistor_SMD:R_0603_1608Metric" (at 183.642 53.34 90)
       (effects (font (size 1.27 1.27)) hide)
     )
@@
       (effects (font (size 1.27 1.27)) (justify left))
     )
-    (property "Footprint" "" (at 53.0352 38.1 0)
+    (property "Footprint" "Capacitor_SMD:C_0603_1608Metric" (at 53.0352 38.1 0)
       (effects (font (size 1.27 1.27)) hide)
     )
@@
       (effects (font (size 1.27 1.27)) (justify left))
     )
-    (property "Footprint" "" (at 121.412 58.42 90)
+    (property "Footprint" "Resistor_SMD:R_0603_1608Metric" (at 121.412 58.42 90)
       (effects (font (size 1.27 1.27)) hide)
     )
@@
       (effects (font (size 1.27 1.27)) (justify left))
     )
-    (property "Footprint" "" (at 35.56 88.9 0)
+    (property "Footprint" "Button_Switch_SMD:SW_SPST_SKQG_WithStem" (at 35.56 88.9 0)
       (effects (font (size 1.27 1.27)) hide)
     )
@@
       (effects (font (size 1.27 1.27)) (justify right))
     )
-    (property "Footprint" "" (at 30.48 165.1 90)
+    (property "Footprint" "Connector_PinHeader_2.54mm:PinHeader_2x03_P2.54mm_Vertical_SMD" (at 30.48 165.1 90)
       (effects (font (size 1.27 1.27)) hide)
     )
@@
       (effects (font (size 1.27 1.27)) (justify left))
     )
-    (property "Footprint" "" (at 149.5552 46.99 0)
+    (property "Footprint" "Capacitor_SMD:C_0603_1608Metric" (at 149.5552 46.99 0)
       (effects (font (size 1.27 1.27)) hide)
     )
@@
       (effects (font (size 1.27 1.27)) (justify left))
     )
-    (property "Footprint" "" (at 162.2552 46.99 0)
+    (property "Footprint" "Capacitor_SMD:C_0603_1608Metric" (at 162.2552 46.99 0)
       (effects (font (size 1.27 1.27)) hide)
     )
@@
       (effects (font (size 1.27 1.27)) (justify left))
     )
-    (property "Footprint" "" (at 256.2352 148.59 0)
+    (property "Footprint" "Capacitor_SMD:C_0805_2012Metric" (at 256.2352 148.59 0)
       (effects (font (size 1.27 1.27)) hide)
     )
@@
       (effects (font (size 1.27 1.27)) (justify right))
     )
-    (property "Footprint" "" (at 139.7 72.39 0)
+    (property "Footprint" "Package_SO:SOIC-8_3.9x4.9mm_P1.27mm" (at 139.7 72.39 0)
       (effects (font (size 1.27 1.27)) hide)
     )
@@
       (effects (font (size 1.27 1.27)) (justify left))
     )
-    (property "Footprint" "" (at 178.1048 95.25 0)
-      (effects (font (size 1.27 1.27)) hide)
-    )
+    (property "Footprint" "Capacitor_SMD:C_0603_1608Metric" (at 178.1048 95.25 0)
+      (effects (font (size 1.27 1.27)) hide)
+    )

Commit message: Touched up schematic and initial layout
Parts:
- removed C3: 10 uF, Capacitor_SMD:C_0603_1608Metric, symbol Device:C
- removed C4: 100 nF, Capacitor_SMD:C_0603_1608Metric, symbol Device:C
- removed R3: 10k, Resistor_SMD:R_0603_1608Metric, symbol Device:R
- removed U1: MCP3426A0T-E/SN, Package_SO:SOIC-8_3.9x4.9mm_P1.27mm, symbol Analog_ADC:MCP3426-xSN
- added C10, C12, C6, C9: 10uF, Capacitor_SMD:C_0805_2012Metric, symbol Device:C
- added C13: 22uF, Capacitor_SMD:C_0805_2012Metric, symbol Device:C
- added C5, C7, C8: 0.1uF, Capacitor_SMD:C_0603_1608Metric, symbol Device:C
- added U3: ~, ADC Pretty:QFN-12_EP_2x2_Pitch0.4mm, symbol Sensor Customs:MCP3465
- added U4: AZ1117-3.3, Package_TO_SOT_SMD:SOT-223-3_TabPin2, symbol Regulator_Linear:AZ1117-3.3
- J4: footprint Connector_AMASS:AMASS_XT60-F_1x02_P7.20mm_Vertical -> Connector_AMASS:AMASS_XT60-M_1x02_P7.20mm_Vertical
- J5: footprint Connector_AMASS:AMASS_XT60-M_1x02_P7.20mm_Vertical -> Connector_AMASS:AMASS_XT60-F_1x02_P7.20mm_Vertical
- R3: renamed from R4; value ? -> 30k
- R4: renamed from R5; value ? -> 10k
- Y1: value 16M -> 8M
- renumbered C7 to C11, C8 to C14, C5 to C3, C6 to C4, X1 to U1, U3 to U5
Connections:
- net +5V: now also C12.1, U4.3 (VI); no longer C1.1, C2.1, R2.1, U1.18 (AVCC), U1.4 (VCC), U1.6 (VCC)
- net BATT_DIVIDED: now also U3.4 (CH1)
- net CURRENT: now also U3.5 (CH0)
- net GND: now also C10.2, C12.2, C13.2, C5.2, C6.2, C7.2, C8.2, C9.2, U3.1 (AGND), U3.10 (DGND), U3.2 (REFIN-), U4.1 (GND)
- net MISO: now also U3.9 (SDO)
- net MOSI: now also U3.8 (SDI)
- net RESET: now also J1.5 (~{RST})
- net SCK: now also U3.7 (SCK)
- net SDA: no longer R2.2
- net SS: no longer J1.5 (~{RST})
- net CS: now reaches U1.12 (PB0)
- net CS: now also R2.1, U3.6 (CS)
- new net: C10.1, C8.1, U3.3 (REFIN+)
- new net +3V3: C1.1, C13.1, C2.1, C5.1, C6.1, C7.1, C9.1, R2.2, U1.18 (AVCC), U1.4 (VCC), U1.6 (VCC), U3.11 (DVDD), U3.12 (AVDD), U4.2 (VO)
- no-connect marks 17 -> 16
Other:
- moved on the sheet: C3, C4, J4, J5, R3, R4, U2
