File: motherboard/motherboard.kicad_sch (KiCad schematic)
At the start: 45 parts, among them J1 Raspberry_Pi_2_3 ANT, J14 USB_C_Receptacle_USB2.0, J2 PROGRAM, J3 Battery / Pitot/ Orientation, J4 c02 censor, J5 shaftencorder, J7 SparLoad, J8 lidar, J9 Control Board, Q1 2N7002K, SW1 MCU_RST, U1 Bluetooth Module - Shaft Power, U2 IMU, U3 Bluetooth Module - Power Cont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, U4 GPS module, U5 DHT11(DHT22), U6 STM32F412RETx, U7 nRF24L01-telemetry-INTERIOR, U8 nRF24L01-telemetry-EXTERIOR, U9 DPS310 - barometer, Y1 8M

Commit message: Edited layout
Parts:
- added H5, H6, H7, H8: MountingHole, MountingHole:MountingHole_2.7mm_M2.5, symbol Mechanical:MountingHole
Changed lines of the file:
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@@
+    )
+  )
+  (symbol (lib_id "Mechanical:MountingHole") (at 95.25 78.74 0) (unit 1)
+    (in_bom yes) (on_board yes) (dnp no) (fields_autoplaced)
+    (property "Reference" "H7" (at 97.79 78.105 0)
+      (effects (font (size 1.27 1.27)) (justify left))
+    )
+    (property "Value" "MountingHole" (at 97.79 80.645 0)
+      (effects (font (size 1.27 1.27)) (justify left))
+    )
+    (property "Footprint" "MountingHole:MountingHole_2.7mm_M2.5" (at 95.25 78.74 0)
+      (effects (font (size 1.27 1.27)) hide)
+    )
+    (property "Datasheet" "~" (at 95.25 78.74 0)
+      (effects (font (size 1.27 1.27)) hide)
+    )
+    (instances
+      (project "motherboard"
+        (path "/39c7ec0f-0a05-4172-b48a-dcc9b63f77ff"
+          (reference "H7") (unit 1)
+        )
+      )
     )
   )
@@
     )
   )
+  (symbol (lib_id "Mechanical:MountingHole") (at 95.25 85.09 0) (unit 1)
+    (in_bom yes) (on_board yes) (dnp no) (fields_autoplaced)
+    (property "Reference" "H6" (at 97.79 84.455 0)
+      (effects (font (size 1.27 1.27)) (justify left))
+    )
+    (property "Value" "MountingHole" (at 97.79 86.995 0)
+      (effects (font (size 1.27 1.27)) (justify left))
+    )
+    (property "Footprint" "MountingHole:MountingHole_2.7mm_M2.5" (at 95.25 85.09 0)
+      (effects (font (size 1.27 1.27)) hide)
+    )
+    (property "Datasheet" "~" (at 95.25 85.09 0)
+      (effects (font (size 1.27 1.27)) hide)
+    )
+    (instances
+      (project "motherboard"
+        (path "/39c7ec0f-0a05-4172-b48a-dcc9b63f77ff"
+          (reference "H6") (unit 1)
+        )
+      )
+    )
+  )
   (symbol (lib_id "Device:C") (at 237.49 54.61 0) (mirror x) (unit 1)
     (in_bom yes) (on_board yes) (dnp no)
@@
         (path "/a202737f-3bef-4789-86fe-0d52089f6e3f"
           (reference "C6") (unit 1)
+        )
+      )
+    )
+  )
+  (symbol (lib_id "Mechanical:MountingHole") (at 95.25 92.71 0) (unit 1)
+    (in_bom yes) (on_board yes) (dnp no) (fields_autoplaced)
+    (property "Reference" "H5" (at 97.79 92.075 0)
+      (effects (font (size 1.27 1.27)) (justify left))
+    )
+    (property "Value" "MountingHole" (at 97.79 94.615 0)
+      (effects (font (size 1.27 1.27)) (justify left))
+    )
+    (property "Footprint" "MountingHole:MountingHole_2.7mm_M2.5" (at 95.25 92.71 0)
+      (effects (font (size 1.27 1.27)) hide)
+    )
+    (property "Datasheet" "~" (at 95.25 92.71 0)
+      (effects (font (size 1.27 1.27)) hide)
+    )
+    (instances
+      (project "motherboard"
+        (path "/39c7ec0f-0a05-4172-b48a-dcc9b63f77ff"
+          (reference "H5") (unit 1)
         )
       )
@@
         )
       )
+    )
+  )
+  (symbol (lib_id "Mechanical:MountingHole") (at 95.25 71.12 0) (unit 1)
+    (in_bom yes) (on_board yes) (dnp no) (fields_autoplaced)
+    (property "Reference" "H8" (at 97.79 70.485 0)
+      (effects (font (size 1.27 1.27)) (justify left))
+    )
+    (property "Value" "MountingHole" (at 97.79 73.025 0)
+      (effects (font (size 1.27 1.27)) (justify left))
+    )
+    (property "Footprint" "MountingHole:MountingHole_2.7mm_M2.5" (at 95.25 71.12 0)
+      (effects (font (size 1.27 1.27)) hide)
+    )
+    (property "Datasheet" "~" (at 95.25 71.12 0)
+      (effects (font (size 1.27 1.27)) hide)
+    )
+    (instances
+      (project "motherboard"
+        (path "/39c7ec0f-0a05-4172-b48a-dcc9b63f77ff"
+          (reference "H8") (unit 1)
+        )
+      )

Commit message: Edited rev2 layout
Parts:
- removed H2: MountingHole, MountingHole:MountingHole_2.5mm_Pad, symbol Mechanical:MountingHole
Changed lines of the file:
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@@
-    )
-  )
-  (symbol (lib_id "Mechanical:MountingHole") (at 327.66 223.52 0) (unit 1)
-    (in_bom yes) (on_board yes) (dnp no) (fields_autoplaced)
-    (property "Reference" "H2" (at 330.2 222.885 0)
-      (effects (font (size 1.27 1.27)) (justify left))
-    )
-    (property "Value" "MountingHole" (at 330.2 225.425 0)
-      (effects (font (size 1.27 1.27)) (justify left))
-    )
-    (property "Footprint" "MountingHole:MountingHole_2.5mm_Pad" (at 327.66 223.52 0)
-      (effects (font (size 1.27 1.27)) hide)
-    )
-    (property "Datasheet" "~" (at 327.66 223.52 0)
-      (effects (font (size 1.27 1.27)) hide)
-    )
-    (instances
-      (project "motherboard"
-        (path "/39c7ec0f-0a05-4172-b48a-dcc9b63f77ff"
-          (reference "H2") (unit 1)
-        )
-      )
     )
   )
