File: prop_pitch_nrf24/prop_pitch_nrf24.kicad_sch (KiCad schematic)
At the start: 55 parts, among them J1 LOAD1, J2 LOAD2, J3 AVR-UPDI-6, J4 SERVO2, J5 SERVO1, J6 SERIAL, Q1 MMSS8550, U1 ATtiny1616-M, U1 TPS563208DDCR, U2 HX711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

Commit message: Revised buck circuit and added symbol
Parts:
- removed C2: 22uF, Capacitor_SMD:C_0805_2012Metric, symbol Device:C
- removed U1: TPS563208DDCR, Package_TO_SOT_SMD:TSOT-23-6, symbol Regulators:TPS563208DDCR
- added U3: TPS563208DDCR, Package_TO_SOT_SMD:TSOT-23-6, symbol TPS563208DDCR:TPS563208DDCR
- C1: value 22uF -> 10u
- C3: value 22uF -> 100n; footprint Capacitor_SMD:C_0805_2012Metric -> Capacitor_SMD:C_0603_1608Metric
- C8, C9: value 22uF -> 22u
- L1: value 3.3uH -> 3u3
- R1: value 54.9k -> 54k9
Connections:
- net EN is gone; now on net +BATT: R3.1
- net +5V: now also L1.2; no longer L1.1
- net +BATT: now also U3.3 (VIN); no longer R3.2
- net GND: now also U3.1 (GND)
- net BST: no longer names the net of C7.2
- net BST: now also L1.1, U3.2 (SW)
- net SW: no longer names the net of C7.1
- net SW: now also U3.6 (VBST); no longer L1.2
- net VFB renamed FB
- net FB: now also U3.4 (VFB)
- new net: R3.2, U3.5 (EN)
