File: control/control.kicad_pcb (KiCad board)
At the start: 2 copper layers, 54.9 x 56.9 mm, 59 parts, among them J1 Conn_01x02_Pin, J3 Conn_01x02_Pin, J4 Conn_01x07_Pin, J5 Conn_ST_STDC14, P1 Conn_01x03_Pin, P2 Conn_01x03_Pin, P3 Conn_01x03_Pin, P4 Conn_01x03_Pin, SW2 SW_Push, U1 STM32F103C8Tx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

Commit message: updated battery & programmer footprints
Parts:
- Battery1: footprint Connector_AMASS:AMASS_XT60-F_1x02_P7.20mm_Vertical -> Connector_AMASS:AMASS_XT60-M_1x02_P7.20mm_Vertical
- renumbered LED4 to 3V3, LED2 to 5V
Changed lines of the file:
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@@
 		(descr "LED SMD 0805 (2012 Metric), square (rectangular) end terminal, IPC_7351 nominal, (Body size source: https://docs.google.com/spreadsheets/d/1BsfQQcO9C6DZCsRaXUlFlo91Tg2WpOkGARC1WS5S8t0/edit?usp=sharing), generated with kicad-footprint-generator")
 		(tags "LED handsolder")
-		(property "Reference" "LED2"
+		(property "Reference" "5V"
 			(at 0 -1.9 0)
 			(layer "F.SilkS")
@@
 		)
 	)
-	(footprint "Connector_AMASS:AMASS_XT60-F_1x02_P7.20mm_Vertical"
+	(footprint "Connector_AMASS:AMASS_XT60-M_1x02_P7.20mm_Vertical"
 		(layer "F.Cu")
 		(at 140.605 105.713268 90)
@@
 		(tags "XT60 female vertical")
 		(property "Reference" "Battery1"
-			(at 4 -4.25 90)
+			(at 3.6 -5.3 -90)
 			(layer "F.SilkS")
 			(hide yes)
@@
 			)
 		)
-		(property "Footprint" "Connector_AMASS:AMASS_XT60-F_1x02_P7.20mm_Vertical"
+		(property "Footprint" "Connector_AMASS:AMASS_XT60-M_1x02_P7.20mm_Vertical"
 			(at 0 0 90)
 			(unlocked yes)
@@
 			(pintype "passive")
 		)
-		(model "${KICAD8_3DMODEL_DIR}/Connector_AMASS.3dshapes/AMASS_XT60-F_1x02_P7.2mm_Vertical.wrl"
+		(model "${KICAD8_3DMODEL_DIR}/Connector_AMASS.3dshapes/AMASS_XT60-M_1x02_P7.2mm_Vertical.wrl"
 			(offset
 				(xyz 0 0 0)
@@
 		(descr "LED SMD 0805 (2012 Metric), square (rectangular) end terminal, IPC_7351 nominal, (Body size source: https://docs.google.com/spreadsheets/d/1BsfQQcO9C6DZCsRaXUlFlo91Tg2WpOkGARC1WS5S8t0/edit?usp=sharing), generated with kicad-footprint-generator")
 		(tags "LED handsolder")
-		(property "Reference" "LED4"
+		(property "Reference" "3V3"
 			(at 0.005 -1.94 0)
 			(layer "F.SilkS")
