File: control/control.kicad_pcb (KiCad board)
At the start: 2 copper layers, 54.9 x 56.9 mm, 59 parts, among them J1 Conn_01x02_Pin, J3 Conn_01x02_Pin, J4 Conn_01x07_Pin, J5 Conn_ST_STDC14, P1 Conn_01x03_Pin, P2 Conn_01x03_Pin, P3 Conn_01x03_Pin, P4 Conn_01x03_Pin, SW2 SW_Push, U1 STM32F103C8Tx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

Commit message: Fixed power LED labelling
Power indication LEDs had their part references changed to labels causing DRC issues and inconsistency in the board.

Fixed the references to be LED# again and added label text for the power lines.
Parts:
- removed 3V3, 5V: LED1, LED_SMD:LED_0805_2012Metric_Pad1.15x1.40mm_HandSolder
- added LED2: LED1, LED_SMD:LED_0805_2012Metric_Pad1.15x1.40mm_HandSolder, F.Cu at (131.9, 78.6)
- added LED4: LED1, LED_SMD:LED_0805_2012Metric_Pad1.15x1.40mm_HandSolder, F.Cu at (150.9, 68.4)
Other:
- board text added: "3V3"
