File: control/v_regs.kicad_sch (KiCad schematic)
At the start: 25 parts, among them J1 Conn_01x02_Pin, J3 Conn_01x02_Pin

Commit message: updated battery & programmer footprints
Parts:
- Battery1: footprint Connector_AMASS:AMASS_XT60-F_1x02_P7.20mm_Vertical -> Connector_AMASS:AMASS_XT60-M_1x02_P7.20mm_Vertical
Changed lines of the file:
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@@
 			)
 		)
-		(property "Footprint" "Connector_AMASS:AMASS_XT60-F_1x02_P7.20mm_Vertical"
+		(property "Footprint" "Connector_AMASS:AMASS_XT60-M_1x02_P7.20mm_Vertical"
 			(at 41.91 153.67 0)
 			(effects
